File: LED_Matrix_PCB/solenoid_board.sch (KiCad schematic (older format))
At the start: 102 parts, among them J2 MCU_LEFT_LEGS, J3 MCU_RIGHT_LEGS

Commit message: Routed 90% of wires, still need to re-order the column pin masking to better complement the routing.
Parts:
- removed LED8_0, LED8_1, LED8_2, LED8_3, LED8_4, LED8_5, LED8_6, LED8_7, LED8_8: Screw-terminal, TerminalBlock:TerminalBlock_bornier-2_P5.08mm, symbol Connector:Screw_Terminal_01x02
Connections:
- net A4: no longer RS-485.2 (~RE~), RS-485.3 (DE)
- net MISO: now also RS-485.2 (~RE~), RS-485.3 (DE)
Changed lines of the file:
@@
 	3450 2700 3450 2600
 Text Label 3450 2600 2    50   ~ 0
-A4
+MISO
 Wire Wire Line
 	3450 3200 3000 3200
@@
 Text Label 6800 2600 2    50   ~ 0
 ROW7
-Text Label 7600 2900 0    50   ~ 0
-MISO
-Text Label 6800 2900 2    50   ~ 0
-ROW8
 Wire Wire Line
 	6800 850  7600 850
@@
 Wire Wire Line
 	6800 2600 7600 2600
-Wire Wire Line
-	6800 2900 7600 2900
 Text Label 5650 3550 0    50   ~ 0
 ROW0
@@
 COL0
 $Comp
-L Connector:Screw_Terminal_01x02 LED8_0
-U 1 1 5E80C508
-P 5450 6050
-F 0 "LED8_0" H 5450 5850 50  0000 C CNN
-F 1 "Screw-terminal" H 5368 5816 50  0001 C CNN
-F 2 "TerminalBlock:TerminalBlock_bornier-2_P5.08mm" H 5450 6050 50  0001 C CNN
-F 3 "~" H 5450 6050 50  0001 C CNN
-	1    5450 6050
-	-1   0    0    1
-$EndComp
-Text Label 5650 5950 0    50   ~ 0
-ROW8
-Text Label 5650 6050 0    50   ~ 0
-COL0
-$Comp
 L Connector:Screw_Terminal_01x02 LED0_1
 U 1 1 5E816204
@@
 COL1
 $Comp
-L Connector:Screw_Terminal_01x02 LED8_1
-U 1 1 5E816244
-P 6000 6050
-F 0 "LED8_1" H 6000 5850 50  0000 C CNN
-F 1 "Screw-terminal" H 5918 5816 50  0001 C CNN
-F 2 "TerminalBlock:TerminalBlock_bornier-2_P5.08mm" H 6000 6050 50  0001 C CNN
-F 3 "~" H 6000 6050 50  0001 C CNN
-	1    6000 6050
-	-1   0    0    1
-$EndComp
-Text Label 6200 5950 0    50   ~ 0
-ROW8
-Text Label 6200 6050 0    50   ~ 0
-COL1
-$Comp
 L Connector:Screw_Terminal_01x02 LED0_2
 U 1 1 5E823F66
@@
 COL2
 $Comp
-L Connector:Screw_Terminal_01x02 LED8_2
-U 1 1 5E823FA6
-P 6550 6050
-F 0 "LED8_2" H 6550 5850 50  0000 C CNN
-F 1 "Screw-terminal" H 6468 5816 50  0001 C CNN
-F 2 "TerminalBlock:TerminalBlock_bornier-2_P5.08mm" H 6550 6050 50  0001 C CNN
-F 3 "~" H 6550 6050 50  0001 C CNN
-	1    6550 6050
-	-1   0    0    1
-$EndComp
-Text Label 6750 5950 0    50   ~ 0
-ROW8
-Text Label 6750 6050 0    50   ~ 0
-COL2
-$Comp
 L Connector:Screw_Terminal_01x02 LED0_3
 U 1 1 5E823FAE
@@
 COL3
 $Comp
-L Connector:Screw_Terminal_01x02 LED8_3
-U 1 1 5E823FEE
-P 7100 6050
-F 0 "LED8_3" H 7100 5850 50  0000 C CNN
-F 1 "Screw-terminal" H 7018 5816 50  0001 C CNN
-F 2 "TerminalBlock:TerminalBlock_bornier-2_P5.08mm" H 7100 6050 50  0001 C CNN
-F 3 "~" H 7100 6050 50  0001 C CNN
-	1    7100 6050
-	-1   0    0    1
-$EndComp
-Text Label 7300 5950 0    50   ~ 0
-ROW8
-Text Label 7300 6050 0    50   ~ 0
-COL3
-$Comp
 L Connector:Screw_Terminal_01x02 LED0_4
 U 1 1 5E84036A
@@
 COL4
 $Comp
-L Connector:Screw_Terminal_01x02 LED8_4
-U 1 1 5E8403AA
-P 7650 6050
-F 0 "LED8_4" H 7650 5850 50  0000 C CNN
-F 1 "Screw-terminal" H 7568 5816 50  0001 C CNN
-F 2 "TerminalBlock:TerminalBlock_bornier-2_P5.08mm" H 7650 6050 50  0001 C CNN
-F 3 "~" H 7650 6050 50  0001 C CNN
-	1    7650 6050
-	-1   0    0    1
-$EndComp
-Text Label 7850 5950 0    50   ~ 0
-ROW8
-Text Label 7850 6050 0    50   ~ 0
-COL4
-$Comp
 L Connector:Screw_Terminal_01x02 LED0_5
 U 1 1 5E8403B2
@@
 COL5
 $Comp
-L Connector:Screw_Terminal_01x02 LED8_5
-U 1 1 5E8403F2
-P 8200 6050
-F 0 "LED8_5" H 8200 5850 50  0000 C CNN
-F 1 "Screw-terminal" H 8118 5816 50  0001 C CNN
-F 2 "TerminalBlock:TerminalBlock_bornier-2_P5.08mm" H 8200 6050 50  0001 C CNN
-F 3 "~" H 8200 6050 50  0001 C CNN
-	1    8200 6050
-	-1   0    0    1
-$EndComp
-Text Label 8400 5950 0    50   ~ 0
-ROW8
-Text Label 8400 6050 0    50   ~ 0
-COL5
-$Comp
 L Connector:Screw_Terminal_01x02 LED0_6
 U 1 1 5E8403FA
@@
 COL6
 $Comp
-L Connector:Screw_Terminal_01x02 LED8_6
-U 1 1 5E84043A
-P 8750 6050
-F 0 "LED8_6" H 8750 5850 50  0000 C CNN
-F 1 "Screw-terminal" H 8668 5816 50  0001 C CNN
-F 2 "TerminalBlock:TerminalBlock_bornier-2_P5.08mm" H 8750 6050 50  0001 C CNN
-F 3 "~" H 8750 6050 50  0001 C CNN
-	1    8750 6050
-	-1   0    0    1
-$EndComp
-Text Label 8950 5950 0    50   ~ 0
-ROW8
-Text Label 8950 6050 0    50   ~ 0
-COL6
-$Comp
 L Connector:Screw_Terminal_01x02 LED0_7
 U 1 1 5E840442
@@
 COL7
 $Comp
-L Connector:Screw_Terminal_01x02 LED8_7
-U 1 1 5E840482
-P 9300 6050
-F 0 "LED8_7" H 9300 5850 50  0000 C CNN
-F 1 "Screw-terminal" H 9218 5816 50  0001 C CNN
-F 2 "TerminalBlock:TerminalBlock_bornier-2_P5.08mm" H 9300 6050 50  0001 C CNN
-F 3 "~" H 9300 6050 50  0001 C CNN
-	1    9300 6050
-	-1   0    0    1
-$EndComp
-Text Label 9500 5950 0    50   ~ 0
-ROW8
-Text Label 9500 6050 0    50   ~ 0
-COL7
-$Comp
 L Connector:Screw_Terminal_01x02 LED0_8
 U 1 1 5E857C20
@@
 Text Label 10050 5750 0    50   ~ 0
 COL8
-$Comp
-L Connector:Screw_Terminal_01x02 LED8_8
-U 1 1 5E857C60
-P 9850 6050
-F 0 "LED8_8" H 9850 5850 50  0000 C CNN
-F 1 "Screw-terminal" H 9768 5816 50  0001 C CNN
-F 2 "TerminalBlock:TerminalBlock_bornier-2_P5.08mm" H 9850 6050 50  0001 C CNN
-F 3 "~" H 9850 6050 50  0001 C CNN
-	1    9850 6050
-	-1   0    0    1
-$EndComp
-Text Label 10050 5950 0    50   ~ 0
-ROW8
-Text Label 10050 6050 0    50   ~ 0
-COL8
 $EndSCHEMATC

Commit message: Placed finishing touches on V1.0
Connections:
- net D10: now also R333.2; no longer R335.2
- net D11: now also R332.2; no longer R336.2
- net D12: now also R331.2; no longer R337.2
- net D13: now also R330.2; no longer R338.2
- net D5: now also R336.2; no longer R332.2
- net D6: now also R335.2; no longer R333.2
- net SCL: now also R337.2; no longer R331.2
- net SDA: now also R338.2; no longer R330.2
Changed lines of the file:
@@
 $EndComp
 Text Label 9300 850  0    50   ~ 0
-SDA
+D13
 Wire Wire Line
 	9300 850  9050 850
@@
 $EndComp
 Text Label 9300 1100 0    50   ~ 0
-SCL
+D12
 Wire Wire Line
 	9300 1100 9050 1100
@@
 $EndComp
 Text Label 9300 1350 0    50   ~ 0
-D5
+D11
 Wire Wire Line
 	9300 1350 9050 1350
@@
 $EndComp
 Text Label 9300 1600 0    50   ~ 0
-D6
+D10
 Wire Wire Line
 	9300 1600 9050 1600
@@
 $EndComp
 Text Label 9300 2100 0    50   ~ 0
-D10
+D6
 Wire Wire Line
 	9300 2100 9050 2100
@@
 $EndComp
 Text Label 9300 2350 0    50   ~ 0
-D11
+D5
 Wire Wire Line
 	9300 2350 9050 2350
@@
 $EndComp
 Text Label 9300 2600 0    50   ~ 0
-D12
+SCL
 Wire Wire Line
 	9300 2600 9050 2600
@@
 $EndComp
 Text Label 9300 2900 0    50   ~ 0
-D13
+SDA
 Wire Wire Line
 	9300 2900 9050 2900

Commit message: Changed footprints for resistors, changed resistor suppliers, and re-routed wires. Need to add mounting holes and clean for ordering.
Parts:
- R10, R11, R330, R331, R332, R333, R334, R335, R336, R337, R338: footprint Resistor_SMD:R_2010_5025Metric_Pad1.52x2.65mm_HandSolder -> Resistor_THT:R_Axial_DIN0309_L9.0mm_D3.2mm_P20.32mm_Horizontal
Changed lines of the file:
@@
 F 0 "R11" V 2950 3200 50  0000 C CNN
 F 1 "10" V 2750 3200 50  0001 C CNN
-F 2 "Resistor_SMD:R_2010_5025Metric_Pad1.52x2.65mm_HandSolder" V 2780 3200 50  0001 C CNN
+F 2 "Resistor_THT:R_Axial_DIN0309_L9.0mm_D3.2mm_P20.32mm_Horizontal" V 2780 3200 50  0001 C CNN
 F 3 "~" H 2850 3200 50  0001 C CNN
 	1    2850 3200
@@
 F 0 "R10" V 2750 2950 50  0000 C CNN
 F 1 "10" V 2734 2950 50  0001 C CNN
-F 2 "Resistor_SMD:R_2010_5025Metric_Pad1.52x2.65mm_HandSolder" V 2780 2950 50  0001 C CNN
+F 2 "Resistor_THT:R_Axial_DIN0309_L9.0mm_D3.2mm_P20.32mm_Horizontal" V 2780 2950 50  0001 C CNN
 F 3 "~" H 2850 2950 50  0001 C CNN
 	1    2850 2950
@@
 F 0 "R330" V 9000 850 50  0000 C CNN
 F 1 "330" V 9016 850 50  0001 C CNN
-F 2 "Resistor_SMD:R_2010_5025Metric_Pad1.52x2.65mm_HandSolder" V 8830 850 50  0001 C CNN
+F 2 "Resistor_THT:R_Axial_DIN0309_L9.0mm_D3.2mm_P20.32mm_Horizontal" V 8830 850 50  0001 C CNN
 F 3 "~" H 8900 850 50  0001 C CNN
 	1    8900 850
@@
 F 0 "R331" V 9000 1100 50  0000 C CNN
 F 1 "330" V 9016 1100 50  0001 C CNN
-F 2 "Resistor_SMD:R_2010_5025Metric_Pad1.52x2.65mm_HandSolder" V 8830 1100 50  0001 C CNN
+F 2 "Resistor_THT:R_Axial_DIN0309_L9.0mm_D3.2mm_P20.32mm_Horizontal" V 8830 1100 50  0001 C CNN
 F 3 "~" H 8900 1100 50  0001 C CNN
 	1    8900 1100
@@
 F 0 "R332" V 9000 1350 50  0000 C CNN
 F 1 "330" V 9016 1350 50  0001 C CNN
-F 2 "Resistor_SMD:R_2010_5025Metric_Pad1.52x2.65mm_HandSolder" V 8830 1350 50  0001 C CNN
+F 2 "Resistor_THT:R_Axial_DIN0309_L9.0mm_D3.2mm_P20.32mm_Horizontal" V 8830 1350 50  0001 C CNN
 F 3 "~" H 8900 1350 50  0001 C CNN
 	1    8900 1350
@@
 F 0 "R333" V 9000 1600 50  0000 C CNN
 F 1 "R" V 9016 1600 50  0001 C CNN
-F 2 "Resistor_SMD:R_2010_5025Metric_Pad1.52x2.65mm_HandSolder" V 8830 1600 50  0001 C CNN
+F 2 "Resistor_THT:R_Axial_DIN0309_L9.0mm_D3.2mm_P20.32mm_Horizontal" V 8830 1600 50  0001 C CNN
 F 3 "~" H 8900 1600 50  0001 C CNN
 	1    8900 1600
@@
 F 0 "R334" V 9000 1850 50  0000 C CNN
 F 1 "R" V 9016 1850 50  0001 C CNN
-F 2 "Resistor_SMD:R_2010_5025Metric_Pad1.52x2.65mm_HandSolder" V 8830 1850 50  0001 C CNN
+F 2 "Resistor_THT:R_Axial_DIN0309_L9.0mm_D3.2mm_P20.32mm_Horizontal" V 8830 1850 50  0001 C CNN
 F 3 "~" H 8900 1850 50  0001 C CNN
 	1    8900 1850
@@
 F 0 "R335" V 9000 2100 50  0000 C CNN
 F 1 "R" V 9016 2100 50  0001 C CNN
-F 2 "Resistor_SMD:R_2010_5025Metric_Pad1.52x2.65mm_HandSolder" V 8830 2100 50  0001 C CNN
+F 2 "Resistor_THT:R_Axial_DIN0309_L9.0mm_D3.2mm_P20.32mm_Horizontal" V 8830 2100 50  0001 C CNN
 F 3 "~" H 8900 2100 50  0001 C CNN
 	1    8900 2100
@@
 F 0 "R336" V 9000 2350 50  0000 C CNN
 F 1 "R" V 9016 2350 50  0001 C CNN
-F 2 "Resistor_SMD:R_2010_5025Metric_Pad1.52x2.65mm_HandSolder" V 8830 2350 50  0001 C CNN
+F 2 "Resistor_THT:R_Axial_DIN0309_L9.0mm_D3.2mm_P20.32mm_Horizontal" V 8830 2350 50  0001 C CNN
 F 3 "~" H 8900 2350 50  0001 C CNN
 	1    8900 2350
@@
 F 0 "R337" V 9000 2600 50  0000 C CNN
 F 1 "R" V 9016 2600 50  0001 C CNN
-F 2 "Resistor_SMD:R_2010_5025Metric_Pad1.52x2.65mm_HandSolder" V 8830 2600 50  0001 C CNN
+F 2 "Resistor_THT:R_Axial_DIN0309_L9.0mm_D3.2mm_P20.32mm_Horizontal" V 8830 2600 50  0001 C CNN
 F 3 "~" H 8900 2600 50  0001 C CNN
 	1    8900 2600
@@
 F 0 "R338" V 9000 2900 50  0000 C CNN
 F 1 "R" V 9016 2900 50  0001 C CNN
-F 2 "Resistor_SMD:R_2010_5025Metric_Pad1.52x2.65mm_HandSolder" V 8830 2900 50  0001 C CNN
+F 2 "Resistor_THT:R_Axial_DIN0309_L9.0mm_D3.2mm_P20.32mm_Horizontal" V 8830 2900 50  0001 C CNN
 F 3 "~" H 8900 2900 50  0001 C CNN
 	1    8900 2900

Commit message: Forgot to close files before pushing.
Parts:
- removed +5V_IN1: MCU_PWR_Supply, TerminalBlock:TerminalBlock_bornier-2_P5.08mm, symbol Connector:Screw_Terminal_01x02
- removed GND1: Conn_01x01_Male, Connector_PinHeader_2.54mm:PinHeader_1x01_P2.54mm_Vertical, symbol Connector:Conn_01x01_Male
- removed LED0_0, LED0_1, LED0_2, LED0_3, LED0_4, LED0_5, LED0_6, LED0_7, LED0_8, LED1_0, LED1_1, LED1_2, LED1_3, LED1_4, LED1_5, LED1_6, LED1_7, LED1_8, LED2_0, LED2_1, LED2_2, LED2_3, LED2_4, LED2_5, LED2_6, LED2_7, LED2_8, LED3_0, LED3_1, LED3_2, LED3_3, LED3_4, LED3_5, LED3_6, LED3_7, LED3_8, LED4_0, LED4_1, LED4_2, LED4_3, LED4_4, LED4_5, LED4_6, LED4_7, LED4_8, LED5_0, LED5_1, LED5_2, LED5_3, LED5_4, LED5_5, LED5_6, LED5_7, LED5_8, LED6_0, LED6_1, LED6_2, LED6_3, LED6_4, LED6_5, LED6_6, LED6_7, LED6_8, LED7_0, LED7_1, LED7_2, LED7_3, LED7_4, LED7_5, LED7_6, LED7_7, LED7_8: Screw-terminal, TerminalBlock:TerminalBlock_bornier-2_P5.08mm, symbol Connector:Screw_Terminal_01x02
- removed R330, R331, R332: 330, Resistor_THT:R_Axial_DIN0309_L9.0mm_D3.2mm_P20.32mm_Horizontal, symbol Device:R
- removed R333, R334, R335, R336, R337, R338: R, Resistor_THT:R_Axial_DIN0309_L9.0mm_D3.2mm_P20.32mm_Horizontal, symbol Device:R
- removed RJ0, RJ1: RJ45, Connector_RJ:RJ45_Amphenol_54602-x08_Horizontal, symbol Connector:RJ45
- added +5VIN1, COMMS0, COMMS1, LED0_0, LED0_1, LED0_2, LED0_3, LED0_4, LED0_5, LED0_6, LED1_0, LED1_1, LED1_2, LED1_3, LED1_4, LED1_5, LED1_6, LED2_0, LED2_1, LED2_2, LED2_3, LED2_4, LED2_5, LED2_6, LED3_0, LED3_1, LED3_2, LED3_3, LED3_4, LED3_5, LED3_6, LED4_0, LED4_1, LED4_2, LED4_3, LED4_4, LED4_5, LED4_6, LED5_0, LED5_1, LED5_2, LED5_3, LED5_4, LED5_5, LED5_6, LED6_0, LED6_1, LED6_2, LED6_3, LED6_4, LED6_5, LED6_6: Conn_01x02, Connector_PinHeader_2.54mm:PinHeader_1x02_P2.54mm_Vertical, symbol Connector_Generic:Conn_01x02
- added FET0, FET1, FET10, FET11, FET12, FET13, FET2, FET3, FET4, FET5, FET6, FET7, FET8, FET9: 2N7000, digikey-footprints:TO-92-3, symbol dk_Transistors-FETs-MOSFETs-Single:2N7000
- added GND1: Conn_01x01, Connector_PinHeader_2.54mm:PinHeader_1x01_P2.54mm_Vertical, symbol Connector_Generic:Conn_01x01
- added R10k0, R10k1, R10k10, R10k11, R10k12, R10k13, R10k2, R10k3, R10k4, R10k5, R10k6, R10k7, R10k8, R10k9: 10k, Resistor_THT:R_Axial_DIN0204_L3.6mm_D1.6mm_P5.08mm_Vertical, symbol Device:R
- added R300, R301, R302, R303, R304, R305, R306, R307, R308, R309, R310, R311, R312, R313: 300, Resistor_THT:R_Axial_DIN0204_L3.6mm_D1.6mm_P5.08mm_Vertical, symbol Device:R
- R10, R11: footprint Resistor_THT:R_Axial_DIN0309_L9.0mm_D3.2mm_P20.32mm_Horizontal -> Resistor_THT:R_Axial_DIN0204_L3.6mm_D1.6mm_P7.62mm_Horizontal
Connections:
- net +5V: now also +5VIN1.2 (Pin_2), FET0.3 (D), FET1.3 (D), FET10.3 (D), FET11.3 (D), FET12.3 (D), FET13.3 (D), FET2.3 (D), FET3.3 (D), FET4.3 (D), FET5.3 (D), FET6.3 (D), FET7.3 (D), FET8.3 (D), FET9.3 (D)
- net A0: now also R10k0.1
- net A1: now also R10k1.1
- net A2: now also R10k2.1
- net A3: now also R10k3.1
- net A4: now also R10k4.1
- net A5: now also R10k5.1
- net COL0: now also LED0_0.1 (Pin_1), LED1_0.1 (Pin_1), LED2_0.1 (Pin_1), LED3_0.1 (Pin_1), LED4_0.1 (Pin_1), LED5_0.1 (Pin_1), LED6_0.1 (Pin_1), R307.2
- net COL1: now also LED0_1.1 (Pin_1), LED1_1.1 (Pin_1), LED2_1.1 (Pin_1), LED3_1.1 (Pin_1), LED4_1.1 (Pin_1), LED5_1.1 (Pin_1), LED6_1.1 (Pin_1), R308.2
- net COL2: now also LED0_2.1 (Pin_1), LED1_2.1 (Pin_1), LED2_2.1 (Pin_1), LED3_2.1 (Pin_1), LED4_2.1 (Pin_1), LED5_2.1 (Pin_1), LED6_2.1 (Pin_1), R309.2
- net COL3: now also LED0_3.1 (Pin_1), LED1_3.1 (Pin_1), LED2_3.1 (Pin_1), LED3_3.1 (Pin_1), LED4_3.1 (Pin_1), LED5_3.1 (Pin_1), LED6_3.1 (Pin_1), R310.2
- net COL4: now also LED0_4.1 (Pin_1), LED1_4.1 (Pin_1), LED2_4.1 (Pin_1), LED3_4.1 (Pin_1), LED4_4.1 (Pin_1), LED5_4.1 (Pin_1), LED6_4.1 (Pin_1), R311.2
- net COL5: now also LED0_5.1 (Pin_1), LED1_5.1 (Pin_1), LED2_5.1 (Pin_1), LED3_5.1 (Pin_1), LED4_5.1 (Pin_1), LED5_5.1 (Pin_1), LED6_5.1 (Pin_1), R312.2
- net COL6: now also LED0_6.1 (Pin_1), LED1_6.1 (Pin_1), LED2_6.1 (Pin_1), LED3_6.1 (Pin_1), LED4_6.1 (Pin_1), LED5_6.1 (Pin_1), LED6_6.1 (Pin_1), R313.2
- net D10: now also R10k10.1
- net D11: now also R10k9.1
- net D12: now also R10k8.1
- net D13: now also R10k7.1
- net D5: now also R10k13.1
- net D6: now also R10k12.1
- net D9: now also R10k11.1
- net GND: now also +5VIN1.1 (Pin_1), GND1.1 (Pin_1)
- net ROW6: now also LED6_0.2 (Pin_2), LED6_1.2 (Pin_2), LED6_2.2 (Pin_2), LED6_3.2 (Pin_2), LED6_4.2 (Pin_2), LED6_5.2 (Pin_2), LED6_6.2 (Pin_2), R306.2; no longer J2.11 (Pin_11)
- net RJ45_4 renamed A
- net A: now also COMMS0.1 (Pin_1), COMMS1.1 (Pin_1)
- net RJ45_5 renamed B
- net B: now also COMMS0.2 (Pin_2), COMMS1.2 (Pin_2)
- new net: FET0.1 (S), R300.1
- new net: FET0.2 (G), R10k0.2
- new net: FET1.1 (S), R301.1
- new net: FET1.2 (G), R10k1.2
- new net: FET2.1 (S), R302.1
- new net: FET2.2 (G), R10k2.2
- new net: FET3.1 (S), R303.1
- new net: FET3.2 (G), R10k3.2
- new net: FET4.1 (S), R304.1
- new net: FET4.2 (G), R10k4.2
- new net: FET5.1 (S), R305.1
- new net: FET5.2 (G), R10k5.2
- new net: FET6.1 (S), R306.1
- new net: FET6.2 (G), R10k6.2
- new net: FET7.1 (S), R307.1
- new net: FET7.2 (G), R10k7.2
- new net: FET8.1 (S), R308.1
- new net: FET8.2 (G), R10k8.2
- new net: FET9.1 (S), R309.1
- new net: FET9.2 (G), R10k9.2
- new net: FET10.1 (S), R310.1
- new net: FET10.2 (G), R10k10.2
- new net: FET11.1 (S), R311.1
- new net: FET11.2 (G), R10k11.2
- new net: FET12.1 (S), R312.1
- new net: FET12.2 (G), R10k12.2
- new net: FET13.1 (S), R313.1
- new net: FET13.2 (G), R10k13.2
- new net A6: R10k6.1
- new net ROW0: LED0_0.2 (Pin_2), LED0_1.2 (Pin_2), LED0_2.2 (Pin_2), LED0_3.2 (Pin_2), LED0_4.2 (Pin_2), LED0_5.2 (Pin_2), LED0_6.2 (Pin_2), R300.2
- new net ROW1: LED1_0.2 (Pin_2), LED1_1.2 (Pin_2), LED1_2.2 (Pin_2), LED1_3.2 (Pin_2), LED1_4.2 (Pin_2), LED1_5.2 (Pin_2), LED1_6.2 (Pin_2), R301.2
- new net ROW2: LED2_0.2 (Pin_2), LED2_1.2 (Pin_2), LED2_2.2 (Pin_2), LED2_3.2 (Pin_2), LED2_4.2 (Pin_2), LED2_5.2 (Pin_2), LED2_6.2 (Pin_2), R302.2
- new net ROW3: LED3_0.2 (Pin_2), LED3_1.2 (Pin_2), LED3_2.2 (Pin_2), LED3_3.2 (Pin_2), LED3_4.2 (Pin_2), LED3_5.2 (Pin_2), LED3_6.2 (Pin_2), R303.2
- new net ROW4: LED4_0.2 (Pin_2), LED4_1.2 (Pin_2), LED4_2.2 (Pin_2), LED4_3.2 (Pin_2), LED4_4.2 (Pin_2), LED4_5.2 (Pin_2), LED4_6.2 (Pin_2), R304.2
- new net ROW5: LED5_0.2 (Pin_2), LED5_1.2 (Pin_2), LED5_2.2 (Pin_2), LED5_3.2 (Pin_2), LED5_4.2 (Pin_2), LED5_5.2 (Pin_2), LED5_6.2 (Pin_2), R305.2
- new net SCK: J2.11 (Pin_11)
- no-connect marks 16 -> 4
